Commit message: fix: urdf

File: ericlab_description/object_description/urdf/display_object/display_object.macro.xacro (robot description, xacro)
@@ -15,5 +15,5 @@
             <visual>
                 <geometry>
-                    <box size="2 2 0.006"/>
+                    <box size="2 2 0.01"/>
                 </geometry>
             </visual>

File: ericlab_gazebo/object_gazebo/urdf/display_object/display_object.gazebo.xacro (robot description, xacro)
@@ -10,6 +10,6 @@
         <visual>
             <plugin name="screen_video_controller" filename="libgazebo_ros_video.so">
-              <height>600</height>
-              <width>1024</width>
+              <height>2064</height>
+              <width>1544</width>
               <topicName>/display_object_topic</topicName>
               <robotNamespace>display_object</robotNamespace>

Commit message: fix: display_object

File: ericlab_description/object_description/urdf/display_object/display_object.macro.xacro (robot description, xacro)
@@ -9,5 +9,5 @@
         <link name="${suffix}_link">
             <inertial>
-                <origin xyz="0.0 1.9 0.0" rpy="0.0 0.0 0.0"/>
+                <origin xyz="0.0 1.4 0.0" rpy="0.0 0.0 0.0"/>
                 <mass value="0.001"/>
                 <inertia ixx="0.01" ixy="0.0" ixz="0.0" iyy="0.01" iyz="0.0" izz="0.01"/>
@@ -15,9 +15,9 @@
             <visual>
                 <geometry>
-                    <box size="2 2 0.01"/>
+                    <box size="1.5 1.5 0.01"/>
                 </geometry>
             </visual>
             <collision>
-                <origin xyz="0.0 1.9 0.0" rpy="0.0 0.0 0.0"/>
+                <origin xyz="0.0 1.4 0.0" rpy="0.0 0.0 0.0"/>
                 <geometry>
                     <box size="0.01 0.01 0.02"/>

Commit message: fix: denso_box

File: ericlab_description/object_description/urdf/display_object/display_object.macro.xacro (robot description, xacro)
@@ -15,5 +15,5 @@
             <visual>
                 <geometry>
-                    <box size="1.5 1.5 0.01"/>
+                    <box size="1.5 1.5 0.005"/>
                 </geometry>
             </visual>

Commit message: world

File: ericlab_description/object_description/urdf/display_object/display_object.macro.xacro (robot description, xacro)
@@ -15,5 +15,5 @@
             <visual>
                 <geometry>
-                    <box size="1.5 1.5 0.005"/>
+                    <box size="2 2 0.005"/>
                 </geometry>
             </visual>

Commit message: fix: disp

File: ericlab_description/object_description/urdf/display_object/display_object.macro.xacro (robot description, xacro)
@@ -15,5 +15,5 @@
             <visual>
                 <geometry>
-                    <box size="1.5 1.5 0.005"/>
+                    <box size="2 2 0.007"/>
                 </geometry>
             </visual>
